File: Arduino_Mega.kicad_pcb (KiCad board)
At the start: 2 copper layers, 101.6 x 53.3 mm, 13 parts, among them P1 Digital, P10 CONN_1, P11 CONN_1, P12 CONN_1, P13 CONN_1, P2 Power, P3 Analog, P4 Analog, P5 PWM, P6 PWM, P7 Communication, P8 CONN_1, P9 CONN_1

Commit message: Netlist and PCB generated
Parts:
- added C1: 100nF, Capacitors_SMD:C_0805_HandSoldering, F.Cu at (141.0, 108.0)
- added D1: POWER_LED, LEDs:LED_0805, F.Cu at (154.2, 131.7)
- added D2: SERVO_POWER_LED, LEDs:LED_0805, F.Cu at (154.2, 131.7)
- added P14: SERVO_OUT_0, Pin_Headers:Pin_Header_Straight_1x03, F.Cu at (161.9, 75.6)
- added P15: SERVO_OUT_1, Pin_Headers:Pin_Header_Straight_1x03, F.Cu at (158.1, 75.6)
- added P16: SERVO_OUT_2, Pin_Headers:Pin_Header_Straight_1x03, F.Cu at (154.3, 75.6)
- added P17: SERVO_OUT_3, Pin_Headers:Pin_Header_Straight_1x03, F.Cu at (150.5, 75.6)
- added P18: SERVO_OUT_4, Pin_Headers:Pin_Header_Straight_1x03, F.Cu at (146.7, 75.6)
- added P19: SERVO_OUT_5, Pin_Headers:Pin_Header_Straight_1x03, F.Cu at (142.9, 75.6)
- added P20: 5V+, Pin_Headers:Pin_Header_Straight_1x01, F.Cu at (154.2, 131.7)
- added P21: 5V-, Pin_Headers:Pin_Header_Straight_1x01, F.Cu at (154.2, 131.7)
- added P22: PSU_TERMINAL_BLOCK, Pin_Headers:Pin_Header_Straight_1x02, F.Cu at (152.4, 99.1)
- added P23: SENOSRS_IN, Pin_Headers:Pin_Header_Straight_2x05, F.Cu at (133.3, 91.4)
- added P24: PSU_VIN, Pin_Headers:Pin_Header_Straight_1x01, F.Cu at (154.2, 131.7)
- added P25: PSU_VIN-, Pin_Headers:Pin_Header_Straight_1x01, F.Cu at (154.2, 131.7)
- added R1: 10k, Resistors_SMD:R_0805_HandSoldering, F.Cu at (154.3, 110.5)
- added R10, R11: 150, Resistors_SMD:R_0805_HandSoldering, F.Cu at (154.2, 131.7)
- added R2, R3, R4, R5, R6, R7, R8, R9: 10k, Resistors_SMD:R_0805_HandSoldering, F.Cu at (154.2, 131.7)
- added SW1: RST, Buttons_Switches_SMD:SW_SPST_REED_CT05-XXXX-G1, F.Cu at (141.0, 111.8)
Connections:
- net /0(Rx0) renamed /Arduino_CON/0(Rx0)
- net /1(Tx0) renamed /Arduino_CON/1(Tx0)
- net /10(**) renamed /Arduino_CON/10(**)
- net /11(**) renamed /Arduino_CON/11(**)
- net /12(**) renamed /Arduino_CON/12(**)
- net /13(**) renamed /Arduino_CON/13(**)
- net /14(Tx3) renamed /Arduino_CON/14(Tx3)
- net /15(Rx3) renamed /Arduino_CON/15(Rx3)
- net /16(Tx2) renamed /Arduino_CON/16(Tx2)
- net /17(Rx2) renamed /Arduino_CON/17(Rx2)
- net /18(Tx1) renamed /Arduino_CON/18(Tx1)
- net /19(Rx1) renamed /Arduino_CON/19(Rx1)
- net /20(SDA) renamed /Arduino_CON/20(SDA)
- net /21(SCL) renamed /Arduino_CON/21(SCL)
- net /22 renamed /Arduino_CON/22
- net /23 renamed /Arduino_CON/23
- net /24 renamed /Arduino_CON/24
- net /25 renamed /Arduino_CON/25
- net /26 renamed /Arduino_CON/26
- net /27 renamed /Arduino_CON/27
- net /28 renamed /Arduino_CON/28
- net /29 renamed /Arduino_CON/29
- net /30 renamed /Arduino_CON/30
- net /31 renamed /Arduino_CON/31
- net /32 renamed /Arduino_CON/32
- net /33 renamed /Arduino_CON/33
- net /34 renamed /Arduino_CON/34
- net /35 renamed /Arduino_CON/35
- net /36 renamed /Arduino_CON/36
- net /37 renamed /Arduino_CON/37
- net /38 renamed /Arduino_CON/38
- net /39 renamed /Arduino_CON/39
- net /40 renamed /Arduino_CON/40
- net /41 renamed /Arduino_CON/41
- net /42 renamed /Arduino_CON/42
- net /43 renamed /Arduino_CON/43
- net /44 renamed /Arduino_CON/44
- net /45 renamed /Arduino_CON/45
- net /46 renamed /Arduino_CON/46
- net /47 renamed /Arduino_CON/47
- net /48 renamed /Arduino_CON/48
- net /49 renamed /Arduino_CON/49
- net /50(MISO) renamed /Arduino_CON/50(MISO)
- net /51(MOSI) renamed /Arduino_CON/51(MOSI)
- net /52(SCK) renamed /Arduino_CON/52(SCK)
- net /53(SS) renamed /Arduino_CON/53(SS)
- net /8(**) renamed /Arduino_CON/8(**)
- net /9(**) renamed /Arduino_CON/9(**)
- net /A0 renamed /Arduino_CON/ADC_IN_0
- net /A10 renamed /Arduino_CON/A10
- net /A11 renamed /Arduino_CON/A11
- net /A12 renamed /Arduino_CON/A12
- net /A13 renamed /Arduino_CON/A13
- net /A14 renamed /Arduino_CON/A14
- net /A15 renamed /Arduino_CON/A15
- net /A9 renamed /Arduino_CON/A9
- net /AREF renamed /Arduino_CON/AREF
- net /IOREF renamed /Arduino_CON/IOREF
- net /SCL renamed /Arduino_CON/SCL
- net /SDA renamed /Arduino_CON/SDA
- net /Vin renamed /Arduino_CON/Vin
- P2 pad 3: /Reset -> RST
- P3 pad 2: /A1 -> /VoltageDivider/ADC1
- P3 pad 3: /A2 -> /VoltageDivider/ADC2
- P3 pad 4: /A3 -> /VoltageDivider/ADC3
- P3 pad 5: /A4 -> /VoltageDivider/ADC4
- P3 pad 6: /A5 -> /VoltageDivider/ADC5
- P3 pad 7: /A6 -> /VoltageDivider/ADC6
- P3 pad 8: /A7 -> /VoltageDivider/ADC7
- P4 pad 1: /A8 -> /VoltageDivider/ADC8
- P6 pad 1: /7(**) -> /Arduino_CON/PWM5
- P6 pad 2: /6(**) -> /Arduino_CON/PWM4
- P6 pad 3: /5(**) -> /Arduino_CON/PWM3
- P6 pad 4: /4(**) -> /Arduino_CON/PWM2
- P6 pad 5: /3(**) -> /Arduino_CON/PWM1
- P6 pad 6: /2(**) -> /Arduino_CON/PWM0

Commit message: bah
Parts:
- removed P12: CONN_1, Socket_Arduino_Mega:Arduino_1pin
- moved P25 50.7 mm to (184.2, 90.8)
- moved P24 48.2 mm to (191.8, 101.6)
- moved D1 47.8 mm to (118.7, 99.7), turned to 270 degrees
- moved R10 44.6 mm to (118.6, 104.9), turned to 90 degrees
- moved D2 43.3 mm to (125.1, 99.7), turned to 270 degrees
- moved P21 43.0 mm to (191.1, 109.9)
- moved R11 39.7 mm to (125.0, 104.9), turned to 90 degrees
- moved P20 39.6 mm to (186.7, 109.2)
- moved R9 36.4 mm to (174.5, 101.6), turned to 270 degrees
- moved R8 35.0 mm to (172.0, 101.6), turned to 270 degrees
- moved R7 33.8 mm to (169.4, 101.6), turned to 270 degrees
- moved P22 33.2 mm to (185.4, 102.2)
- moved R6 32.7 mm to (166.9, 101.6), turned to 270 degrees
- moved R5 31.8 mm to (164.3, 101.6), turned to 270 degrees
- moved R4 31.1 mm to (161.8, 101.6), turned to 270 degrees
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Routing:
- net +5V: track 0.00 -> 12.7 mm
- net /VoltageDivider/ADC0: track 0.00 -> 7.18 mm
- net /Arduino_CON/PWM5: track 0.00 -> 4.70 mm
- net /Arduino_CON/PWM4: track 0.00 -> 4.70 mm
- net /Arduino_CON/PWM3: track 0.00 -> 4.70 mm
- net /Arduino_CON/PWM2: track 0.00 -> 4.70 mm
- net /Arduino_CON/PWM1: track 0.00 -> 4.70 mm
- net /Arduino_CON/PWM0: track 0.00 -> 4.70 mm

Commit message: PCB rev1.0
Parts:
- removed P10, P11, P13: CONN_1, Socket_Arduino_Mega:Arduino_1pin
- removed P22: PSU_TERMINAL_BLOCK, Pin_Headers:Pin_Header_Straight_1x02
- removed P24: PSU_VIN, Pin_Headers:Pin_Header_Straight_1x01
- removed P25: PSU_VIN-, Pin_Headers:Pin_Header_Straight_1x01
- P8: value CONN_1 -> 5V_SERVO_JP; footprint Socket_Arduino_Mega:Arduino_1pin -> Socket_Strips:Socket_Strip_Straight_1x02
- P9: value CONN_1 -> PWR_OUT; footprint Socket_Arduino_Mega:Arduino_1pin -> Socket_Strips:Socket_Strip_Straight_1x02
- R1, R2, R3, R4, R5, R6, R7, R8, R9: moved to B.Cu
- moved P8 46.1 mm to (138.7, 78.2), turned to 180 degrees
- moved P9 33.3 mm to (142.2, 94.7), turned to 270 degrees
- moved P21 32.9 mm to (169.4, 85.1)
- moved R11 32.1 mm to (144.5, 79.5), turned to 270 degrees
- moved R10 28.4 mm to (131.3, 79.5), turned to 270 degrees
- moved P20 25.9 mm to (169.4, 89.9)
- moved D2 24.5 mm to (144.5, 84.8), turned to 90 degrees
- moved R9 22.2 mm to (177.0, 123.7), turned to 90 degrees
- moved R1 22.1 mm to (154.2, 123.7), turned to 90 degrees
- moved R2 22.1 mm to (156.7, 123.7), turned to 90 degrees
- moved R3 22.1 mm to (159.3, 123.7), turned to 90 degrees
- moved R4 22.1 mm to (161.8, 123.7), turned to 90 degrees
- moved R5 22.1 mm to (164.3, 123.7), turned to 90 degrees
- moved R6 22.1 mm to (166.9, 123.7), turned to 90 degrees
- moved R7 22.1 mm to (169.4, 123.7), turned to 90 degrees
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Connections:
- P1 pad 10: /Arduino_CON/47 -> (no net)
- P1 pad 11: /Arduino_CON/44 -> (no net)
- P1 pad 12: /Arduino_CON/45 -> (no net)
- P1 pad 13: /Arduino_CON/42 -> (no net)
- P1 pad 14: /Arduino_CON/43 -> (no net)
- P1 pad 15: /Arduino_CON/40 -> (no net)
- P1 pad 16: /Arduino_CON/41 -> (no net)
- P1 pad 17: /Arduino_CON/38 -> (no net)
- P1 pad 18: /Arduino_CON/39 -> (no net)
- P1 pad 19: /Arduino_CON/36 -> (no net)
- P1 pad 20: /Arduino_CON/37 -> (no net)
- P1 pad 21: /Arduino_CON/34 -> (no net)
- P1 pad 22: /Arduino_CON/35 -> (no net)
- P1 pad 23: /Arduino_CON/32 -> (no net)
- P1 pad 24: /Arduino_CON/33 -> (no net)
- P1 pad 25: /Arduino_CON/30 -> (no net)
- P1 pad 26: /Arduino_CON/31 -> (no net)
- P1 pad 27: /Arduino_CON/28 -> (no net)
- P1 pad 28: /Arduino_CON/29 -> (no net)
- P1 pad 29: /Arduino_CON/26 -> (no net)
- P1 pad 3: /Arduino_CON/52(SCK) -> (no net)
- P1 pad 30: /Arduino_CON/27 -> (no net)
- P1 pad 31: /Arduino_CON/24 -> (no net)
- P1 pad 32: /Arduino_CON/25 -> (no net)
- P1 pad 33: /Arduino_CON/22 -> (no net)
- P1 pad 34: /Arduino_CON/23 -> (no net)
- P1 pad 4: /Arduino_CON/53(SS) -> (no net)
- P1 pad 5: /Arduino_CON/50(MISO) -> (no net)
- P1 pad 6: /Arduino_CON/51(MOSI) -> (no net)
- P1 pad 7: /Arduino_CON/48 -> (no net)
- P1 pad 8: /Arduino_CON/49 -> (no net)
- P1 pad 9: /Arduino_CON/46 -> (no net)
- P14 pad 2: +5V -> 5V_SERVO
- P15 pad 2: +5V -> 5V_SERVO
- P16 pad 2: +5V -> 5V_SERVO
- P17 pad 2: +5V -> 5V_SERVO
- P18 pad 2: +5V -> 5V_SERVO
- P19 pad 2: +5V -> 5V_SERVO
- P2 pad 1: Net-(P2-Pad1) -> (no net)
- P2 pad 2: /Arduino_CON/IOREF -> (no net)
- P2 pad 4: +3V3 -> (no net)
- P2 pad 8: /Arduino_CON/Vin -> (no net)
- P23 pad 10: /VoltageDivider/ADC8 -> /VoltageDivider/ADC4
- P23 pad 2: /VoltageDivider/ADC0 -> /VoltageDivider/ADC8
- P23 pad 3: /VoltageDivider/ADC1 -> /VoltageDivider/ADC0
- P23 pad 4: /VoltageDivider/ADC2 -> /VoltageDivider/ADC7
- P23 pad 5: /VoltageDivider/ADC3 -> /VoltageDivider/ADC1
- P23 pad 6: /VoltageDivider/ADC4 -> /VoltageDivider/ADC6
- P23 pad 7: /VoltageDivider/ADC5 -> /VoltageDivider/ADC2
- P23 pad 8: /VoltageDivider/ADC6 -> /VoltageDivider/ADC5
- P23 pad 9: /VoltageDivider/ADC7 -> /VoltageDivider/ADC3
- P3 pad 1: /Arduino_CON/ADC_IN_0 -> /VoltageDivider/ADC0
- P4 pad 2: /Arduino_CON/A9 -> (no net)
- P4 pad 3: /Arduino_CON/A10 -> (no net)
- P4 pad 4: /Arduino_CON/A11 -> (no net)
- P4 pad 5: /Arduino_CON/A12 -> (no net)
- P4 pad 6: /Arduino_CON/A13 -> (no net)
- P4 pad 7: /Arduino_CON/A14 -> (no net)
- P4 pad 8: /Arduino_CON/A15 -> (no net)
- P5 pad 1: /Arduino_CON/SCL -> (no net)
- P5 pad 10: /Arduino_CON/8(**) -> (no net)
- P5 pad 2: /Arduino_CON/SDA -> (no net)
- P5 pad 3: /Arduino_CON/AREF -> (no net)
- P5 pad 5: /Arduino_CON/13(**) -> (no net)
- P5 pad 6: /Arduino_CON/12(**) -> (no net)
- P5 pad 7: /Arduino_CON/11(**) -> (no net)
- P5 pad 8: /Arduino_CON/10(**) -> (no net)
- P5 pad 9: /Arduino_CON/9(**) -> (no net)
- P6 pad 7: /Arduino_CON/1(Tx0) -> (no net)
- P6 pad 8: /Arduino_CON/0(Rx0) -> (no net)
- P7 pad 1: /Arduino_CON/14(Tx3) -> (no net)
- P7 pad 2: /Arduino_CON/15(Rx3) -> (no net)
- P7 pad 3: /Arduino_CON/16(Tx2) -> (no net)
- P7 pad 4: /Arduino_CON/17(Rx2) -> (no net)
- P7 pad 5: /Arduino_CON/18(Tx1) -> (no net)
- P7 pad 6: /Arduino_CON/19(Rx1) -> (no net)
- P7 pad 7: /Arduino_CON/20(SDA) -> (no net)
- P7 pad 8: /Arduino_CON/21(SCL) -> (no net)
- P8 pad 1: Net-(P8-Pad1) -> 5V_SERVO
- P9 pad 1: Net-(P9-Pad1) -> +5V
- R11 pad 1: +5V -> 5V_SERVO
Routing:
- net +5V: track 12.7 -> 138.8 mm, vias 0 -> 1
- net /VoltageDivider/ADC8: track 0.00 -> 35.4 mm
- net 5V_SERVO: track 0.00 -> 34.9 mm, vias 0 -> 1
- net /VoltageDivider/ADC7: track 0.00 -> 28.1 mm
- net /VoltageDivider/ADC6: track 0.00 -> 22.7 mm
- net /VoltageDivider/ADC1: track 0.00 -> 22.5 mm
- net /VoltageDivider/ADC0: track 7.18 -> 27.8 mm
- net /VoltageDivider/ADC5: track 0.00 -> 17.9 mm
- net /VoltageDivider/ADC2: track 0.00 -> 17.6 mm
- net RST: track 0.00 -> 14.7 mm, vias 0 -> 1
- net /VoltageDivider/ADC4: track 0.00 -> 13.1 mm
- net /VoltageDivider/ADC3: track 0.00 -> 13.1 mm
- net Net-(D2-Pad2): track 0.00 -> 2.93 mm
- net Net-(D1-Pad2): track 0.00 -> 2.93 mm
- added copper zone on B.Cu, net GND
- added copper zone on F.Cu, net GND
Other:
- board size 101.6 x 53.3 mm -> 101.6 x 58.2 mm
