File: voltage_divs.sch (KiCad schematic (older format))
At the start: 9 parts

Commit message: Netlist and PCB generated
Parts:
- R1, R2, R3, R4, R5, R6, R7, R8, R9: footprint (none) -> Resistors_SMD:R_0805_HandSoldering
Changed lines of the file:
@@
 F 0 "R1" H 1380 1170 50  0000 L CNN
 F 1 "10k" H 1380 1110 50  0000 L CNN
-F 2 "" H 1350 1150 50  0000 C CNN
+F 2 "Resistors_SMD:R_0805_HandSoldering" H 1350 1150 50  0001 C CNN
 F 3 "" H 1350 1150 50  0000 C CNN
 	1    1350 1150
@@
 F 0 "R2" H 1630 1170 50  0000 L CNN
 F 1 "10k" H 1630 1110 50  0000 L CNN
-F 2 "" H 1600 1150 50  0000 C CNN
+F 2 "Resistors_SMD:R_0805_HandSoldering" H 1600 1150 50  0001 C CNN
 F 3 "" H 1600 1150 50  0000 C CNN
 	1    1600 1150
@@
 F 0 "R3" H 1880 1170 50  0000 L CNN
 F 1 "10k" H 1880 1110 50  0000 L CNN
-F 2 "" H 1850 1150 50  0000 C CNN
+F 2 "Resistors_SMD:R_0805_HandSoldering" H 1850 1150 50  0001 C CNN
 F 3 "" H 1850 1150 50  0000 C CNN
 	1    1850 1150
@@
 F 0 "R4" H 2130 1170 50  0000 L CNN
 F 1 "10k" H 2130 1110 50  0000 L CNN
-F 2 "" H 2100 1150 50  0000 C CNN
+F 2 "Resistors_SMD:R_0805_HandSoldering" H 2100 1150 50  0001 C CNN
 F 3 "" H 2100 1150 50  0000 C CNN
 	1    2100 1150
@@
 F 0 "R5" H 2380 1170 50  0000 L CNN
 F 1 "10k" H 2380 1110 50  0000 L CNN
-F 2 "" H 2350 1150 50  0000 C CNN
+F 2 "Resistors_SMD:R_0805_HandSoldering" H 2350 1150 50  0001 C CNN
 F 3 "" H 2350 1150 50  0000 C CNN
 	1    2350 1150
@@
 F 0 "R6" H 2630 1170 50  0000 L CNN
 F 1 "10k" H 2630 1110 50  0000 L CNN
-F 2 "" H 2600 1150 50  0000 C CNN
+F 2 "Resistors_SMD:R_0805_HandSoldering" H 2600 1150 50  0001 C CNN
 F 3 "" H 2600 1150 50  0000 C CNN
 	1    2600 1150
@@
 F 0 "R7" H 2880 1170 50  0000 L CNN
 F 1 "10k" H 2880 1110 50  0000 L CNN
-F 2 "" H 2850 1150 50  0000 C CNN
+F 2 "Resistors_SMD:R_0805_HandSoldering" H 2850 1150 50  0001 C CNN
 F 3 "" H 2850 1150 50  0000 C CNN
 	1    2850 1150
@@
 F 0 "R8" H 3130 1170 50  0000 L CNN
 F 1 "10k" H 3130 1110 50  0000 L CNN
-F 2 "" H 3100 1150 50  0000 C CNN
+F 2 "Resistors_SMD:R_0805_HandSoldering" H 3100 1150 50  0001 C CNN
 F 3 "" H 3100 1150 50  0000 C CNN
 	1    3100 1150
@@
 F 0 "R9" H 3380 1170 50  0000 L CNN
 F 1 "10k" H 3380 1110 50  0000 L CNN
-F 2 "" H 3350 1150 50  0000 C CNN
+F 2 "Resistors_SMD:R_0805_HandSoldering" H 3350 1150 50  0001 C CNN
 F 3 "" H 3350 1150 50  0000 C CNN
 	1    3350 1150
@@
 $EndComp
 $Comp
-L +5V #PWR7
+L +5V #PWR01
 U 1 1 57FD7442
 P 1050 850
-F 0 "#PWR7" H 1050 700 50  0001 C CNN
+F 0 "#PWR01" H 1050 700 50  0001 C CNN
 F 1 "+5V" H 1050 990 50  0000 C CNN
 F 2 "" H 1050 850 50  0000 C CNN
