File: Arduino_CON.sch (KiCad schematic (older format))
At the start: 13 parts, among them P1 Digital, P10 CONN_1, P11 CONN_1, P12 CONN_1, P13 CONN_1, P2 Power, P3 Analog, P4 Analog, P5 PWM, P6 PWM, P7 Communication, P8 CONN_1, P9 CONN_1

Commit message: PCB rev1.0
Parts:
- removed P10, P11, P12, P13, P8, P9: CONN_1, Socket_Arduino_Mega:Arduino_1pin, symbol CONN_1
Connections:
- no-connect marks 7 -> 1
Other:
- note removed: "Holes"
- note removed: "Shield for Arduino Mega Rev 3"
Changed lines of the file:
@@
 AREF
 $Comp
-L +5V #PWR022
+L +5V #PWR018
 U 1 1 5519CA9C
 P 4525 1250
-F 0 "#PWR022" H 4525 1340 20  0001 C CNN
+F 0 "#PWR018" H 4525 1340 20  0001 C CNN
 F 1 "+5V" H 4525 1340 30  0000 C CNN
 F 2 "" H 4525 1250 60  0000 C CNN
@@
 $EndComp
 $Comp
-L +3.3V #PWR023
+L +3.3V #PWR019
 U 1 1 5519CAB8
 P 4650 1250
-F 0 "#PWR023" H 4650 1210 30  0001 C CNN
+F 0 "#PWR019" H 4650 1210 30  0001 C CNN
 F 1 "+3.3V" H 4650 1360 30  0000 C CNN
 F 2 "" H 4650 1250 60  0000 C CNN
@@
 $EndComp
 $Comp
-L GND #PWR024
+L GND #PWR020
 U 1 1 5519CC01
 P 5950 2200
-F 0 "#PWR024" H 5950 2200 30  0001 C CNN
+F 0 "#PWR020" H 5950 2200 30  0001 C CNN
 F 1 "GND" H 5950 2130 30  0001 C CNN
 F 2 "" H 5950 2200 60  0000 C CNN
@@
 $EndComp
 $Comp
-L GND #PWR025
+L GND #PWR021
 U 1 1 5519CDF8
 P 4325 6125
-F 0 "#PWR025" H 4325 6125 30  0001 C CNN
+F 0 "#PWR021" H 4325 6125 30  0001 C CNN
 F 1 "GND" H 4325 6055 30  0001 C CNN
 F 2 "" H 4325 6125 60  0000 C CNN
@@
 $EndComp
 $Comp
-L +5V #PWR026
+L +5V #PWR022
 U 1 1 5519D165
 P 6275 4325
-F 0 "#PWR026" H 6275 4415 20  0001 C CNN
+F 0 "#PWR022" H 6275 4415 20  0001 C CNN
 F 1 "+5V" H 6275 4415 30  0000 C CNN
 F 2 "" H 6275 4325 60  0000 C CNN
@@
 	1    0    0    -1
 $EndComp
-Text Notes 3900 575  0    60   ~ 0
-Shield for Arduino Mega Rev 3
 $Comp
 L CONN_18X2 P1
@@
 $EndComp
 $Comp
-L CONN_1 P8
-U 1 1 551BBA20
-P 6250 700
-F 0 "P8" H 6330 700 40  0000 L CNN
-F 1 "CONN_1" H 6250 755 30  0001 C CNN
-F 2 "Socket_Arduino_Mega:Arduino_1pin" H 6250 700 60  0001 C CNN
-F 3 "" H 6250 700 60  0000 C CNN
-	1    6250 700
-	0    -1   -1   0
-$EndComp
-$Comp
-L CONN_1 P9
-U 1 1 551BBB85
-P 6325 700
-F 0 "P9" H 6405 700 40  0000 L CNN
-F 1 "CONN_1" H 6325 755 30  0001 C CNN
-F 2 "Socket_Arduino_Mega:Arduino_1pin" H 6325 700 60  0001 C CNN
-F 3 "" H 6325 700 60  0000 C CNN
-	1    6325 700
-	0    -1   -1   0
-$EndComp
-$Comp
-L CONN_1 P10
-U 1 1 551BBBAB
-P 6400 700
-F 0 "P10" H 6480 700 40  0000 L CNN
-F 1 "CONN_1" H 6400 755 30  0001 C CNN
-F 2 "Socket_Arduino_Mega:Arduino_1pin" H 6400 700 60  0001 C CNN
-F 3 "" H 6400 700 60  0000 C CNN
-	1    6400 700
-	0    -1   -1   0
-$EndComp
-$Comp
-L CONN_1 P11
-U 1 1 551BBBD7
-P 6475 700
-F 0 "P11" H 6555 700 40  0000 L CNN
-F 1 "CONN_1" H 6475 755 30  0001 C CNN
-F 2 "Socket_Arduino_Mega:Arduino_1pin" H 6475 700 60  0001 C CNN
-F 3 "" H 6475 700 60  0000 C CNN
-	1    6475 700
-	0    -1   -1   0
-$EndComp
-$Comp
-L CONN_1 P12
-U 1 1 551BBC10
-P 6550 700
-F 0 "P12" H 6630 700 40  0000 L CNN
-F 1 "CONN_1" H 6550 755 30  0001 C CNN
-F 2 "Socket_Arduino_Mega:Arduino_1pin" H 6550 700 60  0001 C CNN
-F 3 "" H 6550 700 60  0000 C CNN
-	1    6550 700
-	0    -1   -1   0
-$EndComp
-$Comp
-L CONN_1 P13
-U 1 1 551BBC3C
-P 6625 700
-F 0 "P13" H 6705 700 40  0000 L CNN
-F 1 "CONN_1" H 6625 755 30  0001 C CNN
-F 2 "Socket_Arduino_Mega:Arduino_1pin" H 6625 700 60  0001 C CNN
-F 3 "" H 6625 700 60  0000 C CNN
-	1    6625 700
-	0    -1   -1   0
-$EndComp
-NoConn ~ 6250 850
-NoConn ~ 6325 850
-NoConn ~ 6400 850
-NoConn ~ 6475 850
-NoConn ~ 6550 850
-NoConn ~ 6625 850
-Text Notes 6325 975  0    60   ~ 0
-Holes
-$Comp
-L GND #PWR027
+L GND #PWR023
 U 1 1 5519C84C
 P 4775 2200
-F 0 "#PWR027" H 4775 2200 30  0001 C CNN
+F 0 "#PWR023" H 4775 2200 30  0001 C CNN
 F 1 "GND" H 4775 2130 30  0001 C CNN
 F 2 "" H 4775 2200 60  0000 C CNN
@@
 Wire Wire Line
 	5875 1425 6600 1425
-Wire Notes Line
-	6750 1025 6150 1025
-Wire Notes Line
-	6150 1025 6150 475
-Wire Notes Line
-	3875 650  5375 650
-Wire Notes Line
-	5375 650  5375 475
 Wire Wire Line
 	5950 2200 5950 1525
@@
 Text HLabel 4075 3275 0    60   Input ~ 0
 ADC_IN_8
+Wire Notes Line
+	5375 650  5375 475
 $EndSCHEMATC

Commit message: pcb rev2
Parts:
- removed P1: Digital, Socket_Arduino_Mega:Socket_Strip_Arduino_2x18, symbol CONN_18X2
Connections:
- net labels removed: 22, 23, 24, 25, 26, 27, 28, 29, 30, 31, 32, 33, 34, 35, 36, 37, 38, 39, 40, 41, 42, 43, 44, 45, 46, 47, 48, 49, 50(MISO), 51(MOSI), 52(SCK), 53(SS)
- wire segments 97 -> 55
Changed lines of the file:
@@
 LIBS:contrib
 LIBS:valves
+LIBS:borniers
 LIBS:Arduino_Mega-cache
 EELAYER 25 0
@@
 Text Label 4100 3975 0    60   ~ 0
 A15
-Text Label 6050 4675 1    60   ~ 0
-22
-Text Label 5950 4675 1    60   ~ 0
-24
-Text Label 5850 4675 1    60   ~ 0
-26
-Text Label 5750 4675 1    60   ~ 0
-28
-Text Label 5650 4675 1    60   ~ 0
-30
-Text Label 5550 4675 1    60   ~ 0
-32
-Text Label 5450 4675 1    60   ~ 0
-34
-Text Label 5350 4675 1    60   ~ 0
-36
-Text Label 5250 4675 1    60   ~ 0
-38
-Text Label 5150 4675 1    60   ~ 0
-40
-Text Label 5050 4675 1    60   ~ 0
-42
-Text Label 4950 4675 1    60   ~ 0
-44
-Text Label 4850 4675 1    60   ~ 0
-46
-Text Label 4750 4675 1    60   ~ 0
-48
-Text Label 4650 4825 1    60   ~ 0
-50(MISO)
-Text Label 4550 4825 1    60   ~ 0
-52(SCK)
-Text Label 6050 5850 1    60   ~ 0
-23
-Text Label 5950 5850 1    60   ~ 0
-25
-Text Label 5850 5850 1    60   ~ 0
-27
-Text Label 5650 5850 1    60   ~ 0
-31
-Text Label 5750 5850 1    60   ~ 0
-29
-Text Label 5550 5850 1    60   ~ 0
-33
-Text Label 5450 5850 1    60   ~ 0
-35
-Text Label 5350 5850 1    60   ~ 0
-37
-Text Label 5250 5850 1    60   ~ 0
-39
-Text Label 5150 5850 1    60   ~ 0
-41
-Text Label 5050 5850 1    60   ~ 0
-43
-Text Label 4950 5850 1    60   ~ 0
-45
-Text Label 4850 5850 1    60   ~ 0
-47
-Text Label 4750 5850 1    60   ~ 0
-49
-Text Label 4650 6000 1    60   ~ 0
-51(MOSI)
-Text Label 4550 6000 1    60   ~ 0
-53(SS)
 Text Label 6025 3975 0    60   ~ 0
 21(SCL)
@@
 $Comp
 L GND #PWR021
-U 1 1 5519CDF8
-P 4325 6125
-F 0 "#PWR021" H 4325 6125 30  0001 C CNN
-F 1 "GND" H 4325 6055 30  0001 C CNN
-F 2 "" H 4325 6125 60  0000 C CNN
-F 3 "" H 4325 6125 60  0000 C CNN
-	1    4325 6125
-	1    0    0    -1
-$EndComp
-$Comp
-L +5V #PWR022
-U 1 1 5519D165
-P 6275 4325
-F 0 "#PWR022" H 6275 4415 20  0001 C CNN
-F 1 "+5V" H 6275 4415 30  0000 C CNN
-F 2 "" H 6275 4325 60  0000 C CNN
-F 3 "" H 6275 4325 60  0000 C CNN
-	1    6275 4325
-	1    0    0    -1
-$EndComp
-$Comp
-L CONN_18X2 P1
-U 1 1 5519A11D
-P 5250 5225
-F 0 "P1" H 5250 6125 60  0000 C CNN
-F 1 "Digital" V 5250 5225 50  0000 C CNN
-F 2 "Socket_Arduino_Mega:Socket_Strip_Arduino_2x18" H 5250 5075 60  0001 C CNN
-F 3 "" H 5250 5075 60  0000 C CNN
-	1    5250 5225
-	0    -1   1    0
-$EndComp
-$Comp
-L GND #PWR023
 U 1 1 5519C84C
 P 4775 2200
-F 0 "#PWR023" H 4775 2200 30  0001 C CNN
+F 0 "#PWR021" H 4775 2200 30  0001 C CNN
 F 1 "GND" H 4775 2130 30  0001 C CNN
 F 2 "" H 4775 2200 60  0000 C CNN
@@
 $EndComp
 Wire Wire Line
-	4550 4450 4550 4825
-Wire Wire Line
-	4650 4450 4650 4825
-Wire Wire Line
-	4750 4450 4750 4825
-Wire Wire Line
-	4850 4450 4850 4825
-Wire Wire Line
-	4950 4450 4950 4825
-Wire Wire Line
-	5050 4450 5050 4825
-Wire Wire Line
-	5150 4450 5150 4825
-Wire Wire Line
-	5250 4450 5250 4825
-Wire Wire Line
-	5350 4450 5350 4825
-Wire Wire Line
-	5450 4450 5450 4825
-Wire Wire Line
-	5550 4450 5550 4825
-Wire Wire Line
-	5650 4450 5650 4825
-Wire Wire Line
-	5750 4450 5750 4825
-Wire Wire Line
-	5850 4450 5850 4825
-Wire Wire Line
-	5950 4450 5950 4825
-Wire Wire Line
-	6050 4450 6050 4825
-Wire Wire Line
-	5450 5625 5450 6000
-Wire Wire Line
-	5550 5625 5550 6000
-Wire Wire Line
-	5650 5625 5650 6000
-Wire Wire Line
-	5750 5625 5750 6000
-Wire Wire Line
-	5850 5625 5850 6000
-Wire Wire Line
-	5950 5625 5950 6000
-Wire Wire Line
-	6050 5625 6050 6000
-Wire Wire Line
-	5350 5625 5350 6000
-Wire Wire Line
-	4550 5625 4550 6000
-Wire Wire Line
-	4650 5625 4650 6000
-Wire Wire Line
-	4750 5625 4750 6000
-Wire Wire Line
-	4850 5625 4850 6000
-Wire Wire Line
-	4950 5625 4950 6000
-Wire Wire Line
-	5050 5625 5050 6000
-Wire Wire Line
-	5150 5625 5150 6000
-Wire Wire Line
-	5250 5625 5250 6000
-Wire Wire Line
-	4450 4825 4450 4450
-Wire Wire Line
-	4450 5625 4450 6000
-Wire Wire Line
-	6150 4825 6150 4450
-Wire Wire Line
-	6150 5625 6150 6000
-Wire Wire Line
-	4325 4450 4325 6125
-Wire Wire Line
-	4450 4450 4325 4450
-Wire Wire Line
-	4450 6000 4325 6000
-Connection ~ 4325 6000
-Wire Wire Line
-	6150 4450 6275 4450
-Wire Wire Line
-	6150 6000 6275 6000
-Connection ~ 6275 4450
-Wire Wire Line
 	4850 1525 4775 1525
 Wire Wire Line
@@
 	4400 2125 4850 2125
 Wire Wire Line
-	6275 6000 6275 4325
-Wire Wire Line
 	5875 1625 6600 1625
